File: rev2/nzx/kicad-data/nzx.kicad_sch (KiCad schematic)
At the start: 27 parts

Commit message: feat - Added revision2
Parts:
- A1(GUIDE)1: footprint Kailh_Choc_V2:Kailh_Choc_V2 -> Kailh_Choc_V2:Kailh_Choc_V2_24
- S1(BACK)1: footprint Kailh_Choc_V2:Kailh_Choc_V2_24 -> Kailh_Choc_V2:Kailh_Choc_V2
Changed lines of the file:
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@@
 			)
 		)
-		(property "Footprint" "Kailh_Choc_V2:Kailh_Choc_V2"
+		(property "Footprint" "Kailh_Choc_V2:Kailh_Choc_V2_24"
 			(at 186.69 87.63 0)
 			(effects
@@
 			)
 		)
-		(property "Footprint" "Kailh_Choc_V2:Kailh_Choc_V2_24"
+		(property "Footprint" "Kailh_Choc_V2:Kailh_Choc_V2"
 			(at 91.44 29.21 0)
 			(effects
